Commit message: Updated the collision box for the turtlebot to match the new visuals

File: turtlebot3_description/urdf/turtlebot3_burger.urdf.xacro (robot description, xacro)
@@ -18,7 +18,7 @@
     </visual>
     <collision>
-      <origin xyz="-0.032 0 0.070" rpy="0 0 0"/>
+      <origin xyz="-0.092 0 0.080" rpy="0 0 0"/>
       <geometry>
-        <box size="0.140 0.140 0.143"/>
+        <box size="0.270 0.140 0.143"/>
       </geometry>
     </collision>

Commit message: Started integrating the turtlebot simulations with the main simulations.

File: turtlebot3_description/urdf/turtlebot3_burger.urdf.xacro (robot description, xacro)
@@ -18,7 +18,7 @@
     </visual>
     <collision>
-      <origin xyz="-0.092 0 0.080" rpy="0 0 0"/>
+      <origin xyz="0.038 0 0.080" rpy="0 0 0"/>
       <geometry>
-        <box size="0.270 0.140 0.143"/>
+        <box size="0.250 0.140 0.143"/>
       </geometry>
     </collision>
